File: pcb/Mainboard/Mainboard_v3_modular/Mainboard_v3_modular.brd (EAGLE design)
At the start: 100 x 99 mm, 121 parts, among them IC10 LM1117MP-5.0, IC2 74HC595D, IC3 74HC595D, IC4 74HC595D, IC5 74HC595D, J1 HEAD3X2, J2 USB-MINI-B%C, Q1 IRLML2803, Q11 IRLML2803, Q12 IRLML2803, Q15 IRLML2803, Q19 IRLML2803, Q20 IRLML2803, Q22 IRLML2803, Q23 IRLML2803, Q27 IRLML2803, Q28 IRLML2803, Q3 IRLML2803, Q30 IRLML2803, Q35 IRLML2803, Q37 IRLML2803, Q39 IRLML2803, Q4 IRLML2803, Q42 IRLML2803, Q43 IRLML2803, Q45 IRLML2803, Q47 IRLML2803, Q48 IRLML2803, Q5 IRLML2803, Q50 IRLML2803, Q51 IRLML2803, Q53 IRLML2803, Q55 IRLML2803, Q58 IRLML2803, Q61 IRLML2803, Q63 IRLML2803, Q7 IRLML2803, SW1 RESET, U1 ATMEGA328, Y1 16MHz

Commit message: PCB & Datasheets added
Parts:
- removed U$8: WIRELESS-BLUETOOTH-XS3868, diy_modules:WIRELESS-BLUETOOTH-XS3868
- added C6, C7, C8: 0.1uF, MySMD:CAP0805-NP
- added IC1: LM1117MP-5.0, lm1117_10:SOT223
- added JP2, JP3: (no value), pinhead:1X08
- added LED2, LED3, LED4: BLUE, MySMD:LED0805
- added R11, R12, R13, R6, R8: 1k, rcl:M1206
- added R7: 10k, rcl:M1206
- added SJ10, SJ11, SJ4, SJ5, SJ6, SJ7, SJ8, SJ9: (no value), jumper:SJ
- added TP1, TP2, TP3, TP4: TPSQTP14R, testpad:TP14R
- added U$9: CH340G, ch340g:SOIC16
- added U2: HC_05, SerialPortBluetooth:BLUETOOTH_SMD
- added Y2: 16MHz, MySMD2:RESONATOR
Connections:
- removed net 1.8V_OUT: U$8.12
- removed net AGND: U$8.1
- removed net RST: U$8.13
- removed net VBAT: U$8.11
- new net +3V3: C8.1, IC1.2, IC1.4, JP2.1, R7.1, U2.12
- new net CH340_RX: SJ4.1, U$9.3
- new net CH340_TX: SJ5.1, U$9.2
- new net CTS#: TP4.TP, U$9.9
- new net DCD#: TP1.TP, U$9.12
- new net DF_ADKEY_1: JP3.5
- new net DF_ADKEY_2: JP3.4
- new net DF_BUSY: JP3.1
- new net DF_DAC_L: JP2.5
- new net DF_DAC_R: JP2.4
- new net DF_IO_1: JP3.8
- new net DF_IO_2: JP3.6
- new net DF_RX: JP2.2, SJ8.1
- new net DF_SPK_1: JP2.6
- new net DF_SPK_2: JP2.8
- new net DF_TX: JP2.3, SJ9.1
- new net DF_USB+: JP3.3
- new net DF_USB-: JP3.2
- new net DSR#: TP3.TP, U$9.10
- new net HC05_RX: SJ6.1, U2.2
- new net HC05_TX: SJ7.1, U2.1
- new net N$30: U$9.7, Y2.1
- new net N$31: U$9.8, Y2.3
- new net N$32: LED2.2, R11.2
- new net N$33: LED3.2, R12.2
- new net N$34: C6.2, U$9.4
- new net N$35: U$9.15
- new net N$36: U$9.14
- new net N$37: C7.2, U$9.13
- new net N$38: SJ10.1, SJ11.1
- new net N$41: SJ8.2
- new net N$44: R7.2, U2.11
- new net N$47: SJ9.2
- new net N$50: SJ10.2
- new net N$53: SJ11.2
- new net N$56: LED4.2, R13.2
- new net N$59: R13.1
- new net N$60: R12.1
- new net N$62: R11.1
- new net N$63: R8.1
- new net RI#: TP2.TP, U$9.11
- net +5V: now also C6.1, R6.2, U$9.16
- net COM: now also C8.2, IC1.1, JP2.7, JP3.7, LED2.1, LED3.1, LED4.1, U$9.1, U2.13, U2.14, U2.21, U2.22, Y2.2
- net D0/RX: now also SJ5.2
- net D1/TX: now also SJ4.2
- net D8: now also SJ6.2
- net D9: now also SJ7.2
- net GND: no longer U$8.9
- net N$3: now also R8.2
- net N$5: now also U$9.5
- net N$6: now also U$9.6
- net RESET: now also C7.1, R6.1
- net VIN: now also IC1.3
