File: pcb/Mainboard/Mainboard_v3_modular/Mainboard_v3_modular.sch (EAGLE design)
At the start: 121 parts, among them IC10 LM1117MP-5.0, IC2 74HC595D, IC3 74HC595D, IC4 74HC595D, IC5 74HC595D, J1 HEAD3X2, J2 USB-MINI-B%C, Q1 IRLML2803, Q11 IRLML2803, Q12 IRLML2803, Q15 IRLML2803, Q19 IRLML2803, Q20 IRLML2803, Q22 IRLML2803, Q23 IRLML2803, Q27 IRLML2803, Q28 IRLML2803, Q3 IRLML2803, Q30 IRLML2803, Q35 IRLML2803, Q37 IRLML2803, Q39 IRLML2803, Q4 IRLML2803, Q42 IRLML2803, Q43 IRLML2803, Q45 IRLML2803, Q47 IRLML2803, Q48 IRLML2803, Q5 IRLML2803, Q50 IRLML2803, Q51 IRLML2803, Q53 IRLML2803, Q55 IRLML2803, Q58 IRLML2803, Q61 IRLML2803, Q63 IRLML2803, Q7 IRLML2803, SW1 RESET, U1 ATMEGA328, Y1 16MHz

Commit message: PCB & Datasheets added
Parts:
- removed U$8: WIRELESS-BLUETOOTH-XS3868, diy_modules:WIRELESS-BLUETOOTH-XS3868
- added C6, C7, C8: 0.1uF, MySMD:CAP0805-NP
- added IC1: LM1117MP-5.0, lm1117_10:LM1117MP-5.0
- added JP2, JP3: (no value), pinhead:PINHD-1X8
- added LED2, LED3, LED4: BLUE, MySMD:LED0805
- added R11, R12, R13, R6, R8: 1k, rcl:R-EU_M1206
- added R7: 10k, rcl:R-EU_M1206
- added SJ10, SJ11, SJ4, SJ5, SJ6, SJ7, SJ8, SJ9: (no value), jumper:SJ
- added TP1, TP2, TP3, TP4: TPSQTP14R, testpad:TPSQTP14R
- added U$9: CH340G, ch340g:CH340G
- added U2: HC_05, SerialPortBluetooth:HC_05
- added Y2: 16MHz, MySMD2:RESONATORMU
Connections:
- new net +3V3: C8.1, IC1.OUT, JP2.1, R7.1, U2.3V3
- new net CH340_RX: SJ4.1, U$9.RX
- new net CH340_TX: SJ5.1, U$9.TX
- new net CTS#: TP4.TP, U$9.CTS
- new net DCD#: TP1.TP, U$9.DCD
- new net DF_ADKEY_1: JP3.5
- new net DF_ADKEY_2: JP3.4
- new net DF_BUSY: JP3.1
- new net DF_DAC_L: JP2.5
- new net DF_DAC_R: JP2.4
- new net DF_IO_1: JP3.8
- new net DF_IO_2: JP3.6
- new net DF_RX: JP2.2, SJ8.1
- new net DF_SPK_1: JP2.6
- new net DF_SPK_2: JP2.8
- new net DF_TX: JP2.3, SJ9.1
- new net DF_USB+: JP3.3
- new net DF_USB-: JP3.2
- new net DSR#: TP3.TP, U$9.DSR
- new net HC05_RX: SJ6.1, U2.RX
- new net HC05_TX: SJ7.1, U2.TX
- new net N$30: U$9.XI, Y2.1
- new net N$31: U$9.XO, Y2.3
- new net N$32: LED2.AN, R11.2
- new net N$33: LED3.AN, R12.2
- new net N$34: C6.2, U$9.V3
- new net N$35: U$9.RS232
- new net N$36: U$9.RTS
- new net N$37: C7.2, U$9.DTR
- new net N$38: SJ10.1, SJ11.1
- new net N$41: SJ8.2
- new net N$44: R7.2, U2.RST
- new net N$47: SJ9.2
- new net N$50: SJ10.2
- new net N$53: SJ11.2
- new net N$56: LED4.AN, R13.2
- new net N$59: R13.1
- new net N$60: R12.1
- new net N$62: R11.1
- new net N$63: R8.1
- new net RI#: TP2.TP, U$9.RI
- net +5V: now also C6.1, R6.2, U$9.VCC
- net COM: now also C8.2, IC1.GND, JP2.7, JP3.7, LED2.CA, LED3.CA, LED4.CA, U$9.GND, U2.GND, U2.GND1, U2.GND2, U2.NC, Y2.2
- net D0/RX: now also SJ5.2
- net D1/TX: now also SJ4.2
- net D8: now also SJ6.2
- net D9: now also SJ7.2
- net N$3: now also R8.2
- net N$5: now also U$9.D+
- net N$6: now also U$9.D-
- net RESET: now also C7.1, R6.1
- net VIN: now also IC1.IN
Other:
- note added: "+3V3 REG"
- note added: "Arduino D 11 = pinSoftSerial1RX"
- note added: "Arduino Pin 0 = RX"
- note added: "Arduino Pin 1 = TX"
- note added: "Arduino Pin 10 = pinLatch"
- note added: "Arduino Pin 10 = pinSoftSerial1TX"
- note added: "Arduino Pin 11 = pinData"
- note added: "Arduino Pin 12 = pinClock"
- note added: "Arduino Pin 13 = pinOneWire (egal welcher!)"
- note added: "Arduino Pin 14"
- note added: "Arduino Pin 15 = pinSoftSerial2RX"
- note added: "Arduino Pin 16 = pinSoftSerial2TX"
- note added: "Arduino Pin 2 = pinDCF"
- note added: "Arduino Pin 3 ="
- note added: "Arduino Pin 4 ="
- note added: "Arduino Pin 5 ="
- note added: "Arduino Pin 6 ="
- note added: "Arduino Pin 7 ="
- note added: "BLUETOOTH"
- note added: "Bluetooth"
- note added: "DFPlayer Mini"
- note added: "DFPlayer mini"
- note added: "If using multiple software serial ports, only one can receive data at a time."
- note added: "Not all pins on the Leonardo and Micro support change interrupts, so only the following can be used for RX: 8, 9, 10, 11, 14 (MISO), 15 (SCK), 16 (MOSI)."
- note added: "PAM8403"
- note added: "SoftSerial oder AltSoftSerial ?"
- note added: "USB"
- note added: "n.c."
- moved on the sheet: C2, C5, IC2, IC2P, IC3, IC3P, IC4, IC4P, IC5, IC5P, J1, J2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
